Commit message: able to test with odom

File: steer_bot_description/urdf/clay_roller_bot.urdf.xacro (robot description, xacro)
@@ -48,6 +48,6 @@
   <xacro:property name="wheel_mass" value="1" />
   <!-- Steering link dimensions -->
-  <xacro:property name="steer_radius" value="0.3183" />
-  <xacro:property name="steer_thickness" value="0.85" />
+  <xacro:property name="steer_radius" value="0.1" />
+  <xacro:property name="steer_thickness" value="0.2" />
   <xacro:property name="steer_mass" value="1" />
   <!-- Axle positions -->
@@ -75,12 +75,5 @@
   </link>
   <!-- Front wheel and rear steer joints required for ackermann_steering_controller -->
-  <xacro:front_wheel
-    name="front"
-    parent="base"
-    wheel_radius="${wheel_radius}"
-    wheel_thickness="${wheel_thickness}"
-    wheel_mass="${wheel_mass}">
-    <origin xyz="0 0 ${-wheel_radius-steer_offset}" rpy="${-90 * deg_to_rad} 0 0"/>
-  </xacro:front_wheel>
+  <!-- Front steer and rear wheel joints required for ackermann_steering_controller -->
   <xacro:rear_steer
     name="rear"
@@ -94,4 +87,20 @@
     steer_height="${wheel_radius+steer_offset}">
   </xacro:rear_steer>
+  <xacro:rear_wheel
+    name="rear"
+    parent="rear_steer"
+    wheel_radius="${wheel_radius}"
+    wheel_thickness="${wheel_thickness}"
+    wheel_mass="${wheel_mass}">
+    <origin xyz="0 0 ${-wheel_radius-steer_offset}" rpy="${-90 * deg_to_rad} 0 0"/>
+  </xacro:rear_wheel>
+  <xacro:front_wheel
+    name="front"
+    parent="base"
+    wheel_radius="${wheel_radius}"
+    wheel_thickness="${wheel_thickness}"
+    wheel_mass="${wheel_mass}">
+    <origin xyz="${+base_length/2+axle_offset} 0 0" rpy="${-90 * deg_to_rad} 0 0"/>
+  </xacro:front_wheel>
   <!-- Colour -->
   <gazebo reference="base_link">

File: steer_bot_description/urdf/wheel.xacro (robot description, xacro)
@@ -117,3 +117,44 @@
     </gazebo>
   </xacro:macro>
+  <!-- Bicycle model rear wheel link (passive - no transmission) -->
+  <xacro:macro name="rear_wheel"
+    params="
+      name
+      parent
+      wheel_radius
+      wheel_thickness
+      wheel_mass
+      *origin">
+    <link name="${name}_wheel_link">
+      <visual>
+        <origin xyz="0 0 0" rpy="0 0 0"/>
+        <geometry>
+          <cylinder radius="${wheel_radius}" length="${wheel_thickness}"/>
+        </geometry>
+        <material name="yellow" />
+      </visual>
+      <collision>
+        <origin xyz="0 0 0" rpy="0 0 0"/>
+        <geometry>
+          <cylinder radius="${wheel_radius}" length="${wheel_thickness}"/>
+        </geometry>
+      </collision>
+      <xacro:solid_cylinder_inertial
+          rpy="0 0 0" xyz="0 0 0"
+          mass="${wheel_mass}"
+          radius="${wheel_radius}" length="${wheel_thickness}" />
+    </link>
+    <joint name="${name}_wheel_joint" type="continuous">
+      <parent link="${parent}_link"/>
+      <child link="${name}_wheel_link"/>
+      <xacro:insert_block name="origin"/>
+      <axis xyz="0 0 1"/>
+    </joint>
+    <gazebo reference="${name}_wheel_link">
+      <material>Gazebo/Yellow</material>
+    </gazebo>
+    <gazebo reference="${name}_wheel_joint">
+      <provideFeedback>true</provideFeedback>
+    </gazebo>
+  </xacro:macro>
 </robot>

Commit message: got the base_footprint frame

File: steer_bot_description/urdf/clay_roller_bot.urdf.xacro (robot description, xacro)
@@ -30,5 +30,8 @@
         <robotNamespace>${robot_namespace}</robotNamespace>
         <jointName>
-            front_wheel_joint
+            rear_wheel_joint
+        </jointName>
+        <jointName>
+            front_wheel_footprint_joint
         </jointName>
         <updateRate>50</updateRate>
@@ -74,6 +77,12 @@
         x="${base_length}" y="${base_width}" z="${base_height}" />
   </link>
+  <!-- Non rotating forward wheel link -->
+  <link name="base_footprint"/>
+  <joint name="front_wheel_footprint_joint" type="fixed">
+    <parent link="base_link"/>
+    <child link="base_footprint"/>
+    <origin xyz="${+base_length/2+axle_offset} 0 0" rpy="0 0 0"/>
+  </joint>
   <!-- Front wheel and rear steer joints required for ackermann_steering_controller -->
-  <!-- Front steer and rear wheel joints required for ackermann_steering_controller -->
   <xacro:rear_steer
     name="rear"
@@ -87,4 +96,5 @@
     steer_height="${wheel_radius+steer_offset}">
   </xacro:rear_steer>
+  <!-- Passive Joint ! required-->
   <xacro:rear_wheel
     name="rear"

Commit message: update

File: steer_bot_description/urdf/clay_roller_bot.urdf.xacro (robot description, xacro)
@@ -88,8 +88,8 @@
   </link>
   <!-- Non rotating forward wheel link -->
-  <link name="base_footprint"/>
+  <link name="front_footprint"/>
   <joint name="front_wheel_footprint_joint" type="fixed">
     <parent link="base_link"/>
-    <child link="base_footprint"/>
+    <child link="front_footprint"/>
     <origin xyz="${+base_length/2+axle_offset} 0 0" rpy="0 0 0"/>
   </joint>
